File: hardware/icepool-board-motherboard-2021-01.kicad_pcb (KiCad board)
At the start: 4 copper layers, 152 x 96 mm, 120 parts, among them J1 USB_B_Micro, J10 Conn_02x08_Odd_Even, J11 Conn_02x08_Odd_Even, J12 Conn_02x08_Odd_Even, J13 Conn_02x08_Odd_Even, J14 Conn_02x08_Odd_Even, J15 Conn_02x08_Odd_Even, J16 Conn_02x08_Odd_Even, J17 Conn_02x08_Odd_Even, J18 Conn_02x08_Odd_Even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

Commit message: Finished up layout. Ordered boards.
Parts:
- removed C16, C23, C24, C25, C26, C27, C28, C29, C30, C32, C33, C34, C36: 0.1u, Capacitor_SMD:C_0402_1005Metric
- removed C17: DNP, Capacitor_SMD:C_0402_1005Metric
- removed C19, C20, C21, C22: 4.7u, Capacitor_SMD:C_0402_1005Metric
- removed C31, C35: 10u, Capacitor_SMD:C_0805_2012Metric
- removed D2: LED_IND, LED_SMD:LED_0805_2012Metric
- removed H5, H6: MountingHole_Pad, MountingHole:MountingHole_2.2mm_M2_Pad_Via
- removed J5: Conn_02x08_Odd_Even, Connector_PinHeader_2.54mm:PinHeader_2x08_P2.54mm_Horizontal
- removed JP1: CUT_2V5, Jumper:SolderJumper-2_P1.3mm_Bridged_Pad1.0x1.5mm
- removed R14: 1k, Resistor_SMD:R_0402_1005Metric
- removed R15, R16: 100R, Resistor_SMD:R_0402_1005Metric
- removed R17, R18, R19, R20, R31: 10k, Resistor_SMD:R_0402_1005Metric
- removed U6, U7: AP7361C_SOT-89-5, jkiv-library:SOT89-5
- removed U8: iCE40HX8K-BG121(121-Ball_caBGA), jkiv-library:BGA-121_11x11_9.0x9.0mm
- removed X2: ASEM1-12.000MHZ, Oscillator:Oscillator_SMD_Abracon_ASE-4Pin_3.2x2.5mm
Routing:
- net +1V2: track 44.3 -> 0.00 mm, vias 10 -> 0
- net /ice40hx8k-daughter-board/~LED: track 27.4 -> 0.00 mm
- net /ice40hx8k-daughter-board/~RW: track 26.4 -> 0.00 mm, vias 1 -> 0
- net /ice40hx8k-daughter-board/~CS1: track 26.3 -> 0.00 mm, vias 1 -> 0
- net /ice40hx8k-daughter-board/SDI1: track 25.7 -> 0.00 mm, vias 1 -> 0
- net +3V3: track 51.1 -> 27.4 mm, vias 29 -> 14
- net /ice40hx8k-daughter-board/SDO1: track 23.0 -> 0.00 mm, vias 1 -> 0
- net /ice40hx8k-daughter-board/READY: track 20.8 -> 0.00 mm, vias 1 -> 0
- net /ice40hx8k-daughter-board/CDONE: track 17.5 -> 0.00 mm
- net /ice40hx8k-daughter-board/CRESET_B: track 17.0 -> 0.00 mm
- net /ice40hx8k-daughter-board/SCK1: track 13.7 -> 0.00 mm, vias 1 -> 0
- net /ice40hx8k-daughter-board/SCK0: track 13.0 -> 0.00 mm
- net /ice40hx8k-daughter-board/SDI0: track 12.8 -> 0.00 mm
- net /ice40hx8k-daughter-board/~CS0: track 9.50 -> 0.00 mm
- net GND: track 56.0 -> 48.1 mm, vias 268 -> 255
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- removed copper zone on B.Cu, net (none)
- removed copper zone on F.Cu, net (none)
- removed copper zone on In1.Cu, net (none)
- removed copper zone on In2.Cu, net (none)
Other:
- board size 152 x 96 mm -> 152 x 58 mm
- board text removed: "icepool 2021.01 fourside.io"
