File: hardware/icepool-motherboard/icepool-motherboard.kicad_pcb (KiCad board)
At the start: 4 copper layers, 240 x 40.6 mm, 101 parts, among them J1 Micro_SD_Card_Det_Hirose_DM3AT, J14 PoE_OUT, J15 PoE_IN, J16 PWR_ALT_5, J17 PD Program, J2 USB_C_Receptacle, J3 UART, J4 Abracon_ARJM11-502, SW1 ~nRPIBOOT, U1 Compute_Module_4_Functional, U10 STUSB4500QTR, U11 TPS62132, U12 SN74LVC1G14DBV, U2 PoE_TEMP, U3 PSU_TEMP, U4 SN74LVC1G14DBV, U5 CM4_TEMP, U6 TPD4EUSB30, U7 BOARD_TEMP, U8 TPD4EUSB30, U9 TPD4EUSB30

Commit message: Commit prior to stream.
Parts:
- removed H3, H4: M3_MH, MountingHole:MountingHole_2.7mm_M2.5_ISO7380_Pad
- removed J15: PoE_IN, Connector_PinHeader_2.00mm:PinHeader_1x10_P2.00mm_Vertical
- removed J3: UART, Connector_PinHeader_2.54mm:PinHeader_1x04_P2.54mm_Vertical
- removed R26, R27, R28, R29, R30, R31, R32, R33, R34, R35, R36, R37: 22R, Resistor_SMD:R_0402_1005Metric
- removed U2: PoE_TEMP, Package_TO_SOT_THT:TO-92_Inline
- removed U3: PSU_TEMP, Package_TO_SOT_THT:TO-92_Inline
- removed U5: CM4_TEMP, Package_TO_SOT_THT:TO-92_Inline
- removed U6, U8, U9: TPD4EUSB30, Package_SON:USON-10_2.5x1.0mm_P0.5mm
- removed U7: BOARD_TEMP, Package_TO_SOT_THT:TO-92_Inline
- added D4: TPD2EUSB30DRTR, digikey-footprints:SOT-3, F.Cu at (87.5, 50.5)
- added D5: TPD2EUSB30DRTR, digikey-footprints:SOT-3, F.Cu at (83.4, 48.5)
- added D6: TPD2EUSB30DRTR, digikey-footprints:SOT-3, F.Cu at (47.6, 57.4)
- added D7: TPD2EUSB30DRTR, digikey-footprints:SOT-3, F.Cu at (47.6, 59.1)
- added D8: TPD2EUSB30DRTR, digikey-footprints:SOT-3, F.Cu at (47.6, 65.0)
- added D9: TPD2EUSB30DRTR, digikey-footprints:SOT-3, F.Cu at (47.6, 66.7)
- added J10: Node2, jkiv-library:stamp-10x10-P2.0mm_SMD, F.Cu at (221.0, 64.0)
- added J11: Node7, jkiv-library:stamp-10x10-P2.0mm_SMD, F.Cu at (333.0, 64.0)
- added J12: Node3, jkiv-library:stamp-10x10-P2.0mm_SMD, F.Cu at (249.0, 64.0)
- added J13: Node8, jkiv-library:stamp-10x10-P2.0mm_SMD, F.Cu at (361.0, 64.0)
- added J6: Node0, jkiv-library:stamp-10x10-P2.0mm_SMD, F.Cu at (165.0, 64.0)
- added J7: Node5, jkiv-library:stamp-10x10-P2.0mm_SMD, F.Cu at (277.0, 64.0)
- added J8: Node1, jkiv-library:stamp-10x10-P2.0mm_SMD, F.Cu at (193.0, 64.0)
- added J9: Node6, jkiv-library:stamp-10x10-P2.0mm_SMD, F.Cu at (305.0, 64.0)
- added TP1: I0+, TestPoint:TestPoint_Pad_1.0x1.0mm, F.Cu at (87.0, 75.0)
- added TP2: I0+, TestPoint:TestPoint_Pad_1.0x1.0mm, F.Cu at (85.0, 75.0)
- J1: footprint Connector_Card:microSD_HC_Hirose_DM3AT-SF-PEJM5 -> Connector_Card:microSD_HC_Wuerth_693072010801
- J14: value PoE_OUT -> PoE_PWR; footprint Connector_PinHeader_2.00mm:PinHeader_1x10_P2.00mm_Vertical -> jkiv-library:stamp-10x10-P2.0mm_THT
- J2: footprint Connector_USB:USB_C_Plug_Molex_105444 -> Connector_USB:USB_C_Receptacle_Palconn_UTC16-G
- R24: value 22R -> 0.1R; footprint Resistor_SMD:R_0402_1005Metric -> Resistor_SMD:R_Shunt_Vishay_WSKW0612
- SW1: footprint Button_Switch_SMD:SW_SPST_B3U-1000P -> Button_Switch_SMD:SW_SPST_B3U-3100P
- moved R38 204.7 mm to (376.0, 73.0)
- moved R25 202.2 mm to (376.0, 71.0), turned to 180 degrees
- moved R21 137.6 mm to (28.3, 52.2), turned to 90 degrees
- moved R22 134.1 mm to (29.3, 52.2), turned to 90 degrees
- moved R16 131.2 mm to (29.3, 49.4), turned to 90 degrees
- moved C2 130.3 mm to (28.3, 49.4), turned to 90 degrees
- moved SW1 127.1 mm to (25.0, 50.0), turned to 90 degrees
- moved R24 101.7 mm to (86.0, 72.0), turned to 270 degrees
- moved J16 99.2 mm to (169.0, 41.0), turned to 270 degrees
- moved C7 88.1 mm to (85.9, 59.8)
- moved RN1 64.2 mm to (141.5, 50.0), turned to 180 degrees
- moved L1 63.4 mm to (86.0, 63.0), turned to 90 degrees
- moved RN2 57.0 mm to (141.5, 56.8), turned to 180 degrees
- moved U11 54.0 mm to (86.0, 67.5), turned to 270 degrees
- moved OSHW2 32.6 mm to (64.0, 65.0)
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Connections:
- net /12V-3.3V Buck/DEF renamed /PoE / USB PD/DEF
- net /12V-3.3V Buck/FSW renamed /PoE / USB PD/FSW
- net /12V-3.3V Buck/PD_1v2 renamed /PoE / USB PD/PD_1v2
- net /12V-3.3V Buck/PD_2v7 renamed /PoE / USB PD/PD_2v7
- net /12V-3.3V Buck/PD_GOOD renamed /PoE / USB PD/PD_GOOD
- net /12V-3.3V Buck/PD_RST renamed /PoE / USB PD/PD_RST
- net /12V-3.3V Buck/PD_SCL renamed /PoE / USB PD/PD_SCL
- net /12V-3.3V Buck/PD_SDA renamed /PoE / USB PD/PD_SDA
- net /12V-3.3V Buck/PD_VMCU renamed /PoE / USB PD/PD_VMCU
- net /12V-3.3V Buck/PG renamed /PoE / USB PD/PG
- net /12V-3.3V Buck/SW_3v3 renamed /PoE / USB PD/SW_3v3
- net /12V-3.3V Buck/~ALERT renamed /PoE / USB PD/~ALERT
- C11 pad 1: /12V-3.3V Buck/5V -> /PoE / USB PD/5V
- C13 pad 1: /12V-3.3V Buck/5V -> /PoE / USB PD/5V
- J14 pad 1: GND -> /ETH_TD1+
- J14 pad 10: GND -> Earth
- J14 pad 2: GND -> /ETH_TD1-
- J14 pad 3: GND -> /ETH_TD2+
- J14 pad 4: +5V -> /ETH_TD2-
- J14 pad 5: +5V -> /ETH_CT
- J14 pad 6: +5V -> /ETH_TD3+
- J14 pad 7: +5V -> /ETH_TD3-
- J14 pad 8: GND -> /ETH_TD4+
- J14 pad 9: GND -> /ETH_TD4-
- JP2 pad 1: /12V-3.3V Buck/5V -> /PoE / USB PD/5V
- R24 pad 1: /FPGA_~READY~ -> /PoE / USB PD/5V
- R24 pad 2: /FPGA_~READY~ -> Net-(R24-Pad2)
- U11 pad 10: /12V-3.3V Buck/5V -> /PoE / USB PD/5V
- U11 pad 11: /12V-3.3V Buck/5V -> /PoE / USB PD/5V
- U11 pad 12: /12V-3.3V Buck/5V -> /PoE / USB PD/5V
Routing:
- net /CIPO1: track 0.00 -> 231.8 mm
- net /~nRPIBOOT: track 0.00 -> 90.3 mm
- net /Nodes/SCK1: track 0.00 -> 41.9 mm
- net /Nodes/~CS0: track 0.00 -> 40.3 mm
- net /Nodes/~RESET: track 0.00 -> 39.5 mm
- net /Nodes/~CS1: track 0.00 -> 38.1 mm
- net /Nodes/CRESETB: track 0.00 -> 22.1 mm
- net /PoE / USB PD/PD_SDA: track 0.00 -> 20.4 mm
- net /Nodes/SCK0: track 0.00 -> 19.6 mm
- net /Nodes/COPI1: track 0.00 -> 19.5 mm
- net /PoE / USB PD/PD_SCL: track 0.00 -> 18.8 mm
- net /~ETH_LEDR: track 0.00 -> 16.7 mm
- net /ETH_CT: track 0.00 -> 16.2 mm
- net Earth: track 0.00 -> 15.5 mm
- net Net-(J4-Pad13): track 0.00 -> 15.0 mm
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- added copper zone on B.Cu, net GND
Other:
- board size 240 x 40.6 mm -> 360 x 40 mm
- copper layers 4 -> 2
- net class Default: clearance 0.0889 -> 0.1524; trace_width 0.25 -> 0.1524; via_dia 0.8 -> 0.5; via_drill 0.4 -> 0.25
- rule trace_clearance: 0.0889 -> 0.1524
- rule via_min_drill: 0.254 -> 0.25

Commit message: Start of week commit.
Parts:
- removed C1: 1u, Capacitor_SMD:C_0402_1005Metric
- removed C2: 0.1u, Capacitor_SMD:C_0402_1005Metric
- removed D3: ETH_LEDX, LED_SMD:LED_0603_1608Metric
- removed J4: Abracon_ARJM11-502, Connector_RJ:RJ45_Wuerth_7499111446_Horizontal
- removed R16, R21, R22, R23: 1k0, Resistor_SMD:R_0402_1005Metric
- removed RN1, RN2: 22R, Resistor_SMD:R_Array_Convex_4x0402
- removed SW1: ~nRPIBOOT, Button_Switch_SMD:SW_SPST_B3U-3100P
- added R26: 22R, Resistor_SMD:R_0402_1005Metric, F.Cu at (133.3, 67.3)
- added R27: 22R, Resistor_SMD:R_0402_1005Metric, F.Cu at (133.3, 71.9)
- added R28: 22R, Resistor_SMD:R_0402_1005Metric, F.Cu at (133.3, 74.3)
- added R29: 22R, Resistor_SMD:R_0402_1005Metric, F.Cu at (133.3, 75.3)
- added R30: 22R, Resistor_SMD:R_0402_1005Metric, F.Cu at (133.3, 76.3)
- J1: value Micro_SD_Card_Det_Hirose_DM3AT -> Abracon_ARJ139; footprint Connector_Card:microSD_HC_Wuerth_693072010801 -> jkiv-library:RJ45_Abracon_ARJ136; moved to F.Cu
- J14: footprint jkiv-library:stamp-10x10-P2.0mm_THT -> jkiv-library:expansion-18-P2.0mm_SMD
- R1, R17, R2: value 1k0 -> 22R
- moved J16 185.3 mm to (-12.4, 78.8), turned to 0 degrees
- moved J17 97.0 mm to (-22.0, 81.7)
- moved C7 68.3 mm to (144.6, 94.7), turned to 180 degrees
- moved R2 66.7 mm to (133.3, 69.3), turned to 180 degrees
- moved L1 65.1 mm to (144.5, 91.5), turned to 270 degrees
- moved J1 64.8 mm to (49.0, 68.0)
- moved U11 61.7 mm to (144.5, 87.0), turned to 90 degrees
- moved TP2 60.7 mm to (145.5, 79.5), turned to 90 degrees
- moved R24 59.4 mm to (144.5, 82.5), turned to 90 degrees
- moved TP1 56.7 mm to (143.5, 79.5), turned to 90 degrees
- moved R1 56.0 mm to (133.3, 68.3), turned to 180 degrees
- moved R17 54.9 mm to (133.3, 70.9), turned to 180 degrees
- moved U4 32.1 mm to (105.0, 110.5)
- moved OSHW2 31.4 mm to (39.0, 46.0)
- moved U10 8.20 mm to (73.0, 50.0)
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Connections:
- net /CM4_1v8 renamed +1V8
- net /UART_RX renamed Net-(U1-Pad55)
- net /UART_TX renamed Net-(U1-Pad51)
- net Net-(U1-Pad35) renamed /I2C_SCL
- net Net-(U1-Pad36) renamed /I2C_SDA
- C14 pad 1: +3V3 -> /Node_3v3
- D1 pad 2: /CM4_3v3 -> +3V3
- J1 pad 1: /uSD_D2 -> /ETH_CT
- J1 pad 2: /uSD_D3 -> /ETH_TD3-
- J1 pad 3: /uSD_CMD -> /ETH_TD3+
- J1 pad 4: +3V3 -> /ETH_TD2+
- J1 pad 5: /uSD_CLK -> /ETH_TD2-
- J1 pad 6: Net-(C1-Pad2) -> /ETH_CT
- J1 pad 7: /uSD_D0 -> /ETH_CT
- J1 pad 8: /uSD_D1 -> /ETH_TD4+
- J1 pad 9: /uSD_DETB -> /ETH_TD4-
- J10 pad 22: /Nodes/~READY_3 -> Net-(J10-Pad22)
- J10 pad 24: GND -> Net-(J10-Pad24)
- J10 pad 25: GND -> /Nodes/~READY_3
- J10 pad 3: GND -> /Nodes/~CS1
- J10 pad 34: +3V3 -> /Nodes/Node_3v3
- J10 pad 5: /Nodes/~CS1 -> GND
- J10 pad 6: GND -> /Nodes/~READY_2
- J10 pad 7: /Nodes/SCK1 -> GND
- J10 pad 8: GND -> /Nodes/SCK1
- J10 pad 9: /Nodes/~READY_2 -> GND
- J11 pad 22: /Nodes/~READY_7 -> Net-(J11-Pad22)
- J11 pad 23: GND -> Net-(J11-Pad23)
- J11 pad 24: GND -> Net-(J11-Pad24)
- J11 pad 25: GND -> /Nodes/~READY_7
- J11 pad 26: GND -> Net-(J11-Pad26)
- J11 pad 27: GND -> Net-(J11-Pad27)
- J11 pad 28: GND -> Net-(J11-Pad28)
- J11 pad 29: GND -> Net-(J11-Pad29)
- J11 pad 3: GND -> /Nodes/~CS1
- J11 pad 30: GND -> Net-(J11-Pad30)
- J11 pad 31: GND -> Net-(J11-Pad31)
- J11 pad 34: +3V3 -> /Nodes/Node_3v3
- J11 pad 5: /Nodes/~CS1 -> GND
- J11 pad 6: GND -> /Nodes/~READY_6
- J11 pad 7: /Nodes/SCK1 -> GND
- J11 pad 8: GND -> /Nodes/SCK1
- J11 pad 9: /Nodes/~READY_6 -> GND
- J12 pad 22: /Nodes/~READY_4 -> Net-(J12-Pad22)
- J12 pad 23: GND -> Net-(J12-Pad23)
- J12 pad 24: GND -> Net-(J12-Pad24)
- J12 pad 25: GND -> /Nodes/~READY_4
- J12 pad 26: GND -> Net-(J12-Pad26)
- J12 pad 27: GND -> Net-(J12-Pad27)
- J12 pad 28: GND -> Net-(J12-Pad28)
- J12 pad 29: GND -> Net-(J12-Pad29)
- J12 pad 3: GND -> /Nodes/~CS1
- J12 pad 30: GND -> Net-(J12-Pad30)
- J12 pad 31: GND -> Net-(J12-Pad31)
- J12 pad 34: +3V3 -> /Nodes/Node_3v3
- J12 pad 5: /Nodes/~CS1 -> GND
- J12 pad 6: GND -> /Nodes/~READY_3
- J12 pad 7: /Nodes/SCK1 -> GND
- J12 pad 8: GND -> /Nodes/SCK1
- J12 pad 9: /Nodes/~READY_3 -> GND
- J13 pad 22: /Nodes/~READY_INIT -> Net-(J13-Pad22)
- J13 pad 23: GND -> Net-(J13-Pad23)
- J13 pad 24: GND -> Net-(J13-Pad24)
- J13 pad 25: GND -> /Nodes/~READY_INIT
- J13 pad 26: GND -> Net-(J13-Pad26)
- J13 pad 27: GND -> Net-(J13-Pad27)
- J13 pad 28: GND -> Net-(J13-Pad28)
- J13 pad 29: GND -> Net-(J13-Pad29)
- J13 pad 3: GND -> /Nodes/~CS1
- J13 pad 30: GND -> Net-(J13-Pad30)
- J13 pad 31: GND -> Net-(J13-Pad31)
- J13 pad 34: +3V3 -> /Nodes/Node_3v3
- J13 pad 5: /Nodes/~CS1 -> GND
- J13 pad 6: GND -> /Nodes/~READY_7
- J13 pad 7: /Nodes/SCK1 -> GND
- J13 pad 8: GND -> /Nodes/SCK1
- J13 pad 9: /Nodes/~READY_7 -> GND
- J14 pad 1: /ETH_TD1+ -> +5V
- J14 pad 10: Earth -> /PoE_TAP2
- J14 pad 11: GND -> /PoE_TAP3
- J14 pad 12: GND -> /PoE_TAP3
- J14 pad 13: GND -> /PoE_TAP4
- J14 pad 14: GND -> /PoE_TAP4
- J14 pad 15: GND -> Earth
- J14 pad 16: GND -> Earth
- J14 pad 2: /ETH_TD1- -> +5V
- J14 pad 3: /ETH_TD2+ -> GND
- J14 pad 4: /ETH_TD2- -> GND
- J14 pad 5: /ETH_CT -> GND
- J14 pad 6: /ETH_TD3+ -> GND
- J14 pad 7: /ETH_TD3- -> /PoE_TAP1
- J14 pad 8: /ETH_TD4+ -> /PoE_TAP1
- J14 pad 9: /ETH_TD4- -> /PoE_TAP2
- J6 pad 22: /Nodes/~READY_1 -> Net-(J6-Pad22)
- J6 pad 25: GND -> /Nodes/~READY_1
- J6 pad 27: GND -> Net-(J6-Pad27)
- J6 pad 3: GND -> /Nodes/~CS1
- J6 pad 34: +3V3 -> /Nodes/Node_3v3
- J6 pad 5: /Nodes/~CS1 -> GND
- J6 pad 6: GND -> /FPGA_~READY~
- J6 pad 7: /Nodes/SCK1 -> GND
- J6 pad 8: GND -> /Nodes/SCK1
- J6 pad 9: /FPGA_~READY~ -> GND
- J7 pad 22: /Nodes/~READY_5 -> Net-(J7-Pad22)
- J7 pad 23: GND -> Net-(J7-Pad23)
- J7 pad 24: GND -> Net-(J7-Pad24)
- J7 pad 25: GND -> /Nodes/~READY_5
- J7 pad 26: GND -> Net-(J7-Pad26)
- J7 pad 27: GND -> Net-(J7-Pad27)
- J7 pad 28: GND -> Net-(J7-Pad28)
- J7 pad 29: GND -> Net-(J7-Pad29)
- J7 pad 3: GND -> /Nodes/~CS1
- J7 pad 30: GND -> Net-(J7-Pad30)
- J7 pad 31: GND -> Net-(J7-Pad31)
- J7 pad 34: +3V3 -> /Nodes/Node_3v3
- J7 pad 5: /Nodes/~CS1 -> GND
- J7 pad 6: GND -> /Nodes/~READY_4
- J7 pad 7: /Nodes/SCK1 -> GND
- J7 pad 8: GND -> /Nodes/SCK1
- J7 pad 9: /Nodes/~READY_4 -> GND
- J8 pad 22: /Nodes/~READY_2 -> Net-(J8-Pad22)
- J8 pad 24: GND -> Net-(J8-Pad24)
- J8 pad 25: GND -> /Nodes/~READY_2
- J8 pad 3: GND -> /Nodes/~CS1
- J8 pad 34: +3V3 -> /Nodes/Node_3v3
- J8 pad 5: /Nodes/~CS1 -> GND
- J8 pad 6: GND -> /Nodes/~READY_1
- J8 pad 7: /Nodes/SCK1 -> GND
- J8 pad 8: GND -> /Nodes/SCK1
- J8 pad 9: /Nodes/~READY_1 -> GND
- J9 pad 22: /Nodes/~READY_6 -> Net-(J9-Pad22)
- J9 pad 23: GND -> Net-(J9-Pad23)
- J9 pad 24: GND -> Net-(J9-Pad24)
- J9 pad 25: GND -> /Nodes/~READY_6
- J9 pad 26: GND -> Net-(J9-Pad26)
- J9 pad 27: GND -> Net-(J9-Pad27)
- J9 pad 28: GND -> Net-(J9-Pad28)
- J9 pad 29: GND -> Net-(J9-Pad29)
- J9 pad 3: GND -> /Nodes/~CS1
- J9 pad 30: GND -> Net-(J9-Pad30)
- J9 pad 31: GND -> Net-(J9-Pad31)
- J9 pad 34: +3V3 -> /Nodes/Node_3v3
- J9 pad 5: /Nodes/~CS1 -> GND
- J9 pad 6: GND -> /Nodes/~READY_5
- J9 pad 7: /Nodes/SCK1 -> GND
- J9 pad 8: GND -> /Nodes/SCK1
- J9 pad 9: /Nodes/~READY_5 -> GND
- L1 pad 2: +3V3 -> /Node_3v3
- R1 pad 1: /uSD_DETA -> /Nodes/SCK0
- R1 pad 2: +3V3 -> /SCK0
- R17 pad 1: Net-(R17-Pad1) -> /Nodes/~CS0
- R17 pad 2: /CM4_3v3 -> /~CS0
- R2 pad 1: /uSD_DETB -> /Nodes/COPI0
- R2 pad 2: +3V3 -> /COPI0
- R3 pad 2: /CM4_3v3 -> +3V3
- R4 pad 2: /CM4_3v3 -> +3V3
- R5 pad 2: /CM4_3v3 -> +3V3
- R53 pad 1: +3V3 -> /Node_3v3
- R6 pad 2: /CM4_3v3 -> +3V3
- R7 pad 2: /CM4_3v3 -> +3V3
- R8 pad 2: /CM4_3v3 -> +3V3
- U1 pad 15: /~ETH_LEDX -> /ETH_LEDL
- U1 pad 17: /~ETH_LEDR -> /~ETH_LEDL
- U1 pad 19: /~ETH_LEDL -> /~ETH_LEDR
- U1 pad 57: /uSD_CLK -> (no net)
- U1 pad 61: /uSD_D3 -> (no net)
- U1 pad 62: /uSD_CMD -> (no net)
- U1 pad 63: /uSD_D0 -> (no net)
- U1 pad 64: Net-(U1-Pad64) -> (no net)
- U1 pad 67: /uSD_D1 -> (no net)
- U1 pad 68: Net-(U1-Pad68) -> (no net)
- U1 pad 69: /uSD_D2 -> (no net)
- U1 pad 70: Net-(U1-Pad70) -> (no net)
- U1 pad 72: Net-(U1-Pad72) -> (no net)
- U1 pad 73: GND -> (no net)
- U1 pad 75: Net-(R17-Pad1) -> (no net)
- U1 pad 78: /CM4_3v3 -> +3V3
- U1 pad 84: /CM4_3v3 -> +3V3
- U1 pad 86: /CM4_3v3 -> +3V3
- U11 pad 14: +3V3 -> /Node_3v3
- U4 pad 5: /CM4_3v3 -> +3V3
Routing:
- net /CIPO1: track 231.8 -> 64.0 mm
- net /~nRPIBOOT: track 90.3 -> 0.00 mm
- net /ETH_TD1+: track 0.00 -> 73.4 mm
- net /ETH_TD1-: track 0.00 -> 73.0 mm
- net /ETH_TD2-: track 0.00 -> 70.8 mm
- net /ETH_TD2+: track 0.04 -> 70.4 mm
- net /ETH_TD3+: track 0.00 -> 69.7 mm
- net /ETH_TD3-: track 0.00 -> 69.3 mm
- net /ETH_TD4-: track 0.00 -> 67.8 mm
- net /ETH_TD4+: track 0.00 -> 67.4 mm
- net /USB_D+: track 7.28 -> 45.4 mm
- net /USB_D-: track 6.62 -> 43.7 mm
- net /FPGA_CRESETB: track 0.00 -> 23.9 mm, vias 0 -> 2
- net /Nodes/CRESETB: track 22.1 -> 0.00 mm
- net /PoE / USB PD/PD_SDA: track 20.4 -> 0.00 mm
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
Commit message: Prestream commit.
Parts:
- removed C10, C8, C9: 1u, Capacitor_SMD:C_0402_1005Metric
- removed C11: 10u, Capacitor_SMD:C_1210_3225Metric
- removed C12: 3.3u, Capacitor_SMD:C_0805_2012Metric
- removed C13: 0.1u, Capacitor_SMD:C_0805_2012Metric
- removed C14: 22u, Capacitor_SMD:C_1210_3225Metric
- removed C5: 10u, Capacitor_SMD:C_0402_1005Metric
- removed D5: TPD2EUSB30DRTR, digikey-footprints:SOT-3
- removed J14: PoE_PWR, jkiv-library:expansion-18-P2.0mm_SMD
- removed J16: PWR_ALT_5, Connector_PinHeader_2.54mm:PinHeader_1x02_P2.54mm_Vertical
- removed J17: PD Program, Connector_JST:JST_PH_B4B-PH-SM4-TB_1x04-1MP_P2.00mm_Vertical
- removed JP1: FSW, jkiv-library:J_NO_0201_0603Metric
- removed JP2: DEF, jkiv-library:J_NO_0201_0603Metric
- removed L1: 2.2u, Inductor_SMD:L_Vishay_IHLP-1212
- removed R20: 5k1, Resistor_SMD:R_0402_1005Metric
- removed R24: 0.1R, Resistor_SMD:R_Shunt_Vishay_WSKW0612
- removed R38: 22R, Resistor_SMD:R_0402_1005Metric
- removed R46, R47, R48: 4k7, Resistor_SMD:R_0402_1005Metric
- removed R49, R51: 1k0, Resistor_SMD:R_0402_1005Metric
- removed R52: 10k, Resistor_SMD:R_0402_1005Metric
- removed R53: 100k, Resistor_SMD:R_0805_2012Metric
- removed TP1, TP2: I0+, TestPoint:TestPoint_Pad_1.0x1.0mm
- removed U10: STUSB4500QTR, Package_DFN_QFN:QFN-24-1EP_4x4mm_P0.5mm_EP2.7x2.7mm
- removed U11: TPS62132, Package_DFN_QFN:VQFN-16-1EP_3x3mm_P0.5mm_EP1.68x1.68mm_ThermalVias
- removed U12: SN74LVC1G14DBV, Package_TO_SOT_SMD:SOT-23-5
- added C1: 22u, Capacitor_SMD:C_0402_1005Metric, F.Cu at (401.6, 59.0)
- added H3: M3_MH, MountingHole:MountingHole_3.2mm_M3_DIN965_Pad, F.Cu at (378.0, 44.0)
- added H4: M3_MH, MountingHole:MountingHole_3.2mm_M3_DIN965_Pad, F.Cu at (378.0, 74.0)
- added J3: Micro_SD_Card, Connector_Card:microSD_HC_Molex_104031-0811, B.Cu at (124.2, 69.3)
- added R16: 5k1, Resistor_SMD:R_0402_1005Metric, F.Cu at (369.8, 62.8)
- added R21: 1k0, Resistor_SMD:R_0402_1005Metric, F.Cu at (107.6, 71.9)
- added R22: 1k0, Resistor_SMD:R_0402_1005Metric, F.Cu at (106.1, 71.9)
- added U2: Expansion_PoE, jkiv-library:expansion-poe-P2.0mm_SMD, F.Cu at (70.3, 59.0)
- D2: moved to B.Cu
- H1, H2: footprint MountingHole:MountingHole_2.7mm_M2.5_ISO7380_Pad -> MountingHole:MountingHole_3.2mm_M3_DIN965_Pad
- J11: value Node7 -> Node6
- J13: value Node8 -> Node7
- J2: value USB_C_Receptacle -> USB2.0 Type-C
- J7: value Node5 -> Node4
- J9: value Node6 -> Node5
- moved J2 298.1 mm to (378.7, 59.0), turned to 90 degrees
- moved D4 290.6 mm to (371.0, 59.1), turned to 90 degrees
- moved R19 244.2 mm to (369.8, 64.8)
- moved FB1 235.8 mm to (369.6, 68.3)
- moved D2 137.1 mm to (34.4, 41.8), turned to 270 degrees
- moved R18 133.2 mm to (35.0, 44.4), turned to 90 degrees
- moved U4 89.3 mm to (45.9, 43.6), turned to 180 degrees
- moved C7 83.9 mm to (61.0, 88.0), turned to 0 degrees
- moved R8 31.3 mm to (145.5, 104.0)
- moved R9 31.3 mm to (148.4, 103.8)
- moved D1 31.3 mm to (157.8, 91.8)
- moved R10 31.3 mm to (145.5, 98.0)
- moved R11 31.3 mm to (155.6, 96.0)
- moved R12 31.3 mm to (145.5, 102.0)
- moved R14 31.3 mm to (154.2, 98.0)
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Connections:
- net /USB_SBU1 renamed Net-(J2-PadA8)
- net /USB_SBU2 renamed Net-(J2-PadB8)
- J1 pad 17: /~ETH_LEDR -> +3V3
- J10 pad 10: /Nodes/SDO1_1 -> Net-(J10-Pad10)
- J10 pad 11: GND -> Net-(J10-Pad11)
- J10 pad 12: GND -> Net-(J10-Pad12)
- J10 pad 13: GND -> Net-(J10-Pad13)
- J10 pad 14: GND -> Net-(J10-Pad14)
- J10 pad 15: GND -> Net-(J10-Pad15)
- J10 pad 16: GND -> Net-(J10-Pad16)
- J10 pad 17: GND -> Net-(J10-Pad17)
- J10 pad 18: GND -> Net-(J10-Pad18)
- J10 pad 19: GND -> Net-(J10-Pad19)
- J10 pad 20: GND -> Net-(J10-Pad20)
- J10 pad 21: /Nodes/SDO1_2 -> Net-(J10-Pad21)
- J10 pad 26: GND -> /Nodes/SDO1_2
- J10 pad 33: Net-(J10-Pad33) -> +5V
- J10 pad 34: /Nodes/Node_3v3 -> Net-(J10-Pad34)
- J10 pad 4: GND -> /Nodes/SCK1
- J10 pad 5: GND -> /Nodes/SDO1_1
- J10 pad 7: GND -> Net-(J10-Pad7)
- J10 pad 8: /Nodes/SCK1 -> Net-(J10-Pad8)
- J10 pad 9: GND -> Net-(J10-Pad9)
- J11 pad 10: /Nodes/SDO1_5 -> Net-(J11-Pad10)
- J11 pad 11: GND -> Net-(J11-Pad11)
- J11 pad 12: GND -> Net-(J11-Pad12)
- J11 pad 13: GND -> Net-(J11-Pad13)
- J11 pad 14: GND -> Net-(J11-Pad14)
- J11 pad 15: GND -> Net-(J11-Pad15)
- J11 pad 16: GND -> Net-(J11-Pad16)
- J11 pad 17: GND -> Net-(J11-Pad17)
- J11 pad 18: GND -> Net-(J11-Pad18)
- J11 pad 19: GND -> Net-(J11-Pad19)
- J11 pad 20: GND -> Net-(J11-Pad20)
- J11 pad 21: /Nodes/SDO1_6 -> Net-(J11-Pad21)
- J11 pad 26: Net-(J11-Pad26) -> /Nodes/SDO1_6
- J11 pad 31: Net-(J11-Pad31) -> GND
- J11 pad 33: Net-(J11-Pad33) -> +5V
- J11 pad 34: /Nodes/Node_3v3 -> Net-(J11-Pad34)
- J11 pad 4: GND -> /Nodes/SCK1
- J11 pad 5: GND -> /Nodes/SDO1_5
- J11 pad 7: GND -> Net-(J11-Pad7)
- J11 pad 8: /Nodes/SCK1 -> Net-(J11-Pad8)
- J11 pad 9: GND -> Net-(J11-Pad9)
- J12 pad 10: /Nodes/SDO1_2 -> Net-(J12-Pad10)
- J12 pad 11: GND -> Net-(J12-Pad11)
- J12 pad 12: GND -> Net-(J12-Pad12)
- J12 pad 13: GND -> Net-(J12-Pad13)
- J12 pad 14: GND -> Net-(J12-Pad14)
- J12 pad 15: GND -> Net-(J12-Pad15)
- J12 pad 16: GND -> Net-(J12-Pad16)
- J12 pad 17: GND -> Net-(J12-Pad17)
- J12 pad 18: GND -> Net-(J12-Pad18)
- J12 pad 19: GND -> Net-(J12-Pad19)
- J12 pad 20: GND -> Net-(J12-Pad20)
- J12 pad 21: /Nodes/SDO1_3 -> Net-(J12-Pad21)
- J12 pad 26: Net-(J12-Pad26) -> /Nodes/SDO1_3
- J12 pad 31: Net-(J12-Pad31) -> GND
- J12 pad 33: Net-(J12-Pad33) -> +5V
- J12 pad 34: /Nodes/Node_3v3 -> Net-(J12-Pad34)
- J12 pad 4: GND -> /Nodes/SCK1
- J12 pad 5: GND -> /Nodes/SDO1_2
- J12 pad 7: GND -> Net-(J12-Pad7)
- J12 pad 8: /Nodes/SCK1 -> Net-(J12-Pad8)
- J12 pad 9: GND -> Net-(J12-Pad9)
- J13 pad 10: /Nodes/SDO1_6 -> Net-(J13-Pad10)
- J13 pad 11: GND -> Net-(J13-Pad11)
- J13 pad 12: GND -> Net-(J13-Pad12)
- J13 pad 13: GND -> Net-(J13-Pad13)
- J13 pad 14: GND -> Net-(J13-Pad14)
- J13 pad 15: GND -> Net-(J13-Pad15)
- J13 pad 16: GND -> Net-(J13-Pad16)
- J13 pad 17: GND -> Net-(J13-Pad17)
- J13 pad 18: GND -> Net-(J13-Pad18)
- J13 pad 19: GND -> Net-(J13-Pad19)
- J13 pad 20: GND -> Net-(J13-Pad20)
- J13 pad 21: /CIPO1 -> Net-(J13-Pad21)
- J13 pad 25: /Nodes/~READY_INIT -> /Nodes/CIPO1
- J13 pad 31: Net-(J13-Pad31) -> GND
- J13 pad 33: Net-(J13-Pad33) -> +5V
- J13 pad 34: /Nodes/Node_3v3 -> Net-(J13-Pad34)
- J13 pad 4: GND -> /Nodes/SCK1
- J13 pad 5: GND -> /Nodes/SDO1_6
- J13 pad 7: GND -> Net-(J13-Pad7)
- J13 pad 8: /Nodes/SCK1 -> Net-(J13-Pad8)
- J13 pad 9: GND -> Net-(J13-Pad9)
- J2 pad A5: /USB_CC1 -> Net-(J2-PadA5)
- J2 pad B5: /USB_CC2 -> Net-(J2-PadB5)
- J6 pad 10: /Nodes/COPI1 -> Net-(J6-Pad10)
- J6 pad 11: GND -> Net-(J6-Pad11)
- J6 pad 12: GND -> Net-(J6-Pad12)
- J6 pad 13: GND -> Net-(J6-Pad13)
- J6 pad 14: GND -> Net-(J6-Pad14)
- J6 pad 15: GND -> Net-(J6-Pad15)
- J6 pad 16: GND -> Net-(J6-Pad16)
- J6 pad 17: GND -> Net-(J6-Pad17)
- J6 pad 18: GND -> Net-(J6-Pad18)
- J6 pad 19: GND -> Net-(J6-Pad19)
- J6 pad 20: GND -> Net-(J6-Pad20)
- J6 pad 21: /Nodes/SDO1_0 -> Net-(J6-Pad21)
- J6 pad 26: Net-(J6-Pad26) -> /Nodes/SDO1_0
- J6 pad 33: Net-(J6-Pad33) -> +5V
- J6 pad 34: /Nodes/Node_3v3 -> Net-(J6-Pad34)
- J6 pad 4: GND -> /Nodes/SCK1
- J6 pad 5: GND -> /Nodes/COPI1
- J6 pad 7: GND -> Net-(J6-Pad7)
- J6 pad 8: /Nodes/SCK1 -> Net-(J6-Pad8)
- J6 pad 9: GND -> Net-(J6-Pad9)
- J7 pad 10: /Nodes/SDO1_3 -> Net-(J7-Pad10)
- J7 pad 11: GND -> Net-(J7-Pad11)
- J7 pad 12: GND -> Net-(J7-Pad12)
- J7 pad 13: GND -> Net-(J7-Pad13)
- J7 pad 14: GND -> Net-(J7-Pad14)
- J7 pad 15: GND -> Net-(J7-Pad15)
- J7 pad 16: GND -> Net-(J7-Pad16)
- J7 pad 17: GND -> Net-(J7-Pad17)
- J7 pad 18: GND -> Net-(J7-Pad18)
- J7 pad 19: GND -> Net-(J7-Pad19)
- J7 pad 20: GND -> Net-(J7-Pad20)
- J7 pad 21: /Nodes/SDO1_4 -> Net-(J7-Pad21)
- J7 pad 26: Net-(J7-Pad26) -> /Nodes/SDO1_4
- J7 pad 31: Net-(J7-Pad31) -> GND
- J7 pad 33: Net-(J7-Pad33) -> +5V
- J7 pad 34: /Nodes/Node_3v3 -> Net-(J7-Pad34)
- J7 pad 4: GND -> /Nodes/SCK1
- J7 pad 5: GND -> /Nodes/~READY_4
- J7 pad 6: /Nodes/~READY_4 -> /Nodes/SDO1_3
- J7 pad 7: GND -> Net-(J7-Pad7)
- J7 pad 8: /Nodes/SCK1 -> Net-(J7-Pad8)
- J7 pad 9: GND -> Net-(J7-Pad9)
- J8 pad 10: /Nodes/SDO1_0 -> Net-(J8-Pad10)
- J8 pad 11: GND -> Net-(J8-Pad11)
- J8 pad 12: GND -> Net-(J8-Pad12)
- J8 pad 13: GND -> Net-(J8-Pad13)
- J8 pad 14: GND -> Net-(J8-Pad14)
- J8 pad 15: GND -> Net-(J8-Pad15)
- J8 pad 16: GND -> Net-(J8-Pad16)
- J8 pad 17: GND -> Net-(J8-Pad17)
- J8 pad 18: GND -> Net-(J8-Pad18)
- J8 pad 19: GND -> Net-(J8-Pad19)
- J8 pad 20: GND -> Net-(J8-Pad20)
- J8 pad 21: /Nodes/SDO1_1 -> Net-(J8-Pad21)
- J8 pad 26: GND -> /Nodes/SDO1_1
- J8 pad 33: Net-(J8-Pad33) -> +5V
- J8 pad 34: /Nodes/Node_3v3 -> Net-(J8-Pad34)
- J8 pad 4: GND -> /Nodes/SCK1
- J8 pad 5: GND -> /Nodes/SDO1_0
- J8 pad 7: GND -> Net-(J8-Pad7)
- J8 pad 8: /Nodes/SCK1 -> Net-(J8-Pad8)
- J8 pad 9: GND -> Net-(J8-Pad9)
- J9 pad 10: /Nodes/SDO1_4 -> Net-(J9-Pad10)
- J9 pad 11: GND -> Net-(J9-Pad11)
- J9 pad 12: GND -> Net-(J9-Pad12)
- J9 pad 13: GND -> Net-(J9-Pad13)
- J9 pad 14: GND -> Net-(J9-Pad14)
- J9 pad 15: GND -> Net-(J9-Pad15)
- J9 pad 16: GND -> Net-(J9-Pad16)
- J9 pad 17: GND -> Net-(J9-Pad17)
- J9 pad 18: GND -> Net-(J9-Pad18)
- J9 pad 19: GND -> Net-(J9-Pad19)
- J9 pad 20: GND -> Net-(J9-Pad20)
- J9 pad 21: /Nodes/SDO1_5 -> Net-(J9-Pad21)
- J9 pad 26: Net-(J9-Pad26) -> /Nodes/SDO1_5
- J9 pad 31: Net-(J9-Pad31) -> GND
- J9 pad 33: Net-(J9-Pad33) -> +5V
- J9 pad 34: /Nodes/Node_3v3 -> Net-(J9-Pad34)
- J9 pad 4: GND -> /Nodes/SCK1
- J9 pad 5: GND -> /Nodes/SDO1_4
- J9 pad 7: GND -> Net-(J9-Pad7)
- J9 pad 8: /Nodes/SCK1 -> Net-(J9-Pad8)
- J9 pad 9: GND -> Net-(J9-Pad9)
- R19 pad 2: /USB_CC1 -> Net-(J2-PadB5)
- R25 pad 2: /Nodes/~READY_INIT -> Net-(J13-Pad26)
- U1 pad 57: (no net) -> /SD_CLK
- U1 pad 61: (no net) -> /SD_DAT3
- U1 pad 62: (no net) -> /SD_CMD
- U1 pad 63: (no net) -> /SD_DAT0
- U1 pad 64: (no net) -> Net-(U1-Pad64)
- U1 pad 67: (no net) -> /SD_DAT1
- U1 pad 68: (no net) -> Net-(U1-Pad68)
- U1 pad 69: (no net) -> /SD_DAT2
- U1 pad 70: (no net) -> Net-(U1-Pad70)
- U1 pad 72: (no net) -> Net-(U1-Pad72)
- U1 pad 73: (no net) -> Net-(U1-Pad73)
- U1 pad 75: (no net) -> /SD_PON
Routing:
- net +5V: track 0.00 -> 393.6 mm
- net /USB_D-: track 43.7 -> 260.9 mm
- net /USB_D+: track 45.4 -> 260.4 mm
- net +3V3: track 0.00 -> 130.3 mm, vias 0 -> 1
- net Net-(J1-Pad18): track 0.00 -> 93.0 mm
- net GND: track 21.9 -> 95.6 mm, vias 28 -> 49
- net /~ETH_LEDL: track 0.00 -> 69.3 mm, vias 0 -> 2
- net Net-(J1-Pad20): track 0.00 -> 61.3 mm, vias 0 -> 1
- net /CIPO1: track 64.0 -> 2.86 mm
- net /Nodes/COPI0: track 0.00 -> 55.6 mm
- net /Nodes/SCK0: track 0.00 -> 48.8 mm
- net Earth: track 0.00 -> 38.1 mm
- net /Nodes/CRESETB: track 0.00 -> 34.2 mm, vias 0 -> 2
- net /PoE_TAP4: track 0.00 -> 31.1 mm
- net /PoE_TAP2: track 0.00 -> 28.6 mm
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