File: hardware/icepool-motherboard/icepool-motherboard.kicad_pcb (KiCad board)
At the start: 2 copper layers, 360 x 40 mm, 66 parts, among them J1 Abracon_ARJ139, J10 Node2, J11 Node6, J12 Node3, J13 Node7, J2 USB2.0 Type-C, J3 Micro_SD_Card, J6 Node0, J7 Node4, J8 Node1, J9 Node5, U1 Compute_Module_4_Functional, U2 Expansion_PoE, U4 SN74LVC1G14DBV

Commit message: Post-stream commit.
* Vertical daughterboards to reduce board size and complexity.
* Flip-flopping on design choices, but meh.
Parts:
- removed J13: Node7, jkiv-library:stamp-10x10-P2.0mm_SMD
- removed U2: Expansion_PoE, jkiv-library:expansion-poe-P2.0mm_SMD
- added J4: DP1435 PoE Module, jkiv-library:DP1435_Module, F.Cu at (64.0, 75.5)
- added J5: Node 0, Connector_PinHeader_2.00mm:PinHeader_1x18_P2.00mm_Vertical_SMD_Pin1Left, F.Cu at (149.0, 59.0)
- C1: footprint Capacitor_SMD:C_0402_1005Metric -> Capacitor_SMD:C_0805_2012Metric
- D2: moved to F.Cu
- J10: value Node2 -> Node 6; footprint jkiv-library:stamp-10x10-P2.0mm_SMD -> Connector_PinHeader_2.00mm:PinHeader_1x18_P2.00mm_Vertical_SMD_Pin1Left
- J11: value Node6 -> Node 3; footprint jkiv-library:stamp-10x10-P2.0mm_SMD -> Connector_PinHeader_2.00mm:PinHeader_1x18_P2.00mm_Vertical_SMD_Pin1Left
- J12: value Node3 -> Node 7; footprint jkiv-library:stamp-10x10-P2.0mm_SMD -> Connector_PinHeader_2.00mm:PinHeader_1x18_P2.00mm_Vertical_SMD_Pin1Left
- J6: value Node0 -> Node 4; footprint jkiv-library:stamp-10x10-P2.0mm_SMD -> Connector_PinHeader_2.00mm:PinHeader_1x18_P2.00mm_Vertical_SMD_Pin1Left
- J7: value Node4 -> Node 1; footprint jkiv-library:stamp-10x10-P2.0mm_SMD -> Connector_PinHeader_2.00mm:PinHeader_1x18_P2.00mm_Vertical_SMD_Pin1Left
- J8: value Node1 -> Node 5; footprint jkiv-library:stamp-10x10-P2.0mm_SMD -> Connector_PinHeader_2.00mm:PinHeader_1x18_P2.00mm_Vertical_SMD_Pin1Left
- J9: value Node5 -> Node 2; footprint jkiv-library:stamp-10x10-P2.0mm_SMD -> Connector_PinHeader_2.00mm:PinHeader_1x18_P2.00mm_Vertical_SMD_Pin1Left
- moved R25 143.1 mm to (223.0, 45.8), turned to 90 degrees
- moved J11 142.9 mm to (179.0, 59.0), turned to 180 degrees
- moved C1 140.8 mm to (260.9, 65.0)
- moved J9 125.0 mm to (169.0, 59.0), turned to 180 degrees
- moved H3 110.0 mm to (268.0, 44.0)
- moved H4 110.0 mm to (268.0, 74.0)
- moved J2 110.0 mm to (268.7, 59.0)
- moved FB1 108.9 mm to (260.8, 62.9)
- moved D4 107.8 mm to (263.2, 58.8)
- moved J7 107.0 mm to (159.0, 59.0), turned to 180 degrees
- moved R19 106.8 mm to (263.3, 57.3)
- moved R16 106.6 mm to (263.2, 60.3)
- moved R22 54.2 mm to (57.0, 49.0)
- moved R21 53.7 mm to (59.0, 49.0)
- moved OSHW2 36.0 mm to (72.7, 69.4)
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Connections:
- J10 pad 1: /Nodes/~CS0 -> +5V
- J10 pad 10: Net-(J10-Pad10) -> /Nodes/SCK1
- J10 pad 11: Net-(J10-Pad11) -> /Nodes/~CS1
- J10 pad 12: Net-(J10-Pad12) -> /Nodes/SDO1_5
- J10 pad 13: Net-(J10-Pad13) -> /Nodes/SDO1_6
- J10 pad 14: Net-(J10-Pad14) -> GND
- J10 pad 15: Net-(J10-Pad15) -> /Nodes/~RESET
- J10 pad 16: Net-(J10-Pad16) -> /Nodes/~READY_6
- J10 pad 17: Net-(J10-Pad17) -> /Nodes/~READY_7
- J10 pad 18: Net-(J10-Pad18) -> GND
- J10 pad 2: /Nodes/~RESET -> GND
- J10 pad 3: /Nodes/~CS1 -> /FPGA_CDONE
- J10 pad 4: /Nodes/SCK1 -> /Nodes/CRESETB
- J10 pad 5: /Nodes/SDO1_1 -> GND
- J10 pad 6: /Nodes/~READY_2 -> /Nodes/SCK0
- J10 pad 7: Net-(J10-Pad7) -> /Nodes/~CS0
- J10 pad 8: Net-(J10-Pad8) -> /Nodes/COPI0
- J10 pad 9: Net-(J10-Pad9) -> GND
- J11 pad 1: /Nodes/~CS0 -> +5V
- J11 pad 10: Net-(J11-Pad10) -> /Nodes/SCK1
- J11 pad 11: Net-(J11-Pad11) -> /Nodes/~CS1
- J11 pad 12: Net-(J11-Pad12) -> /Nodes/SDO1_2
- J11 pad 13: Net-(J11-Pad13) -> /Nodes/SDO1_3
- J11 pad 14: Net-(J11-Pad14) -> GND
- J11 pad 15: Net-(J11-Pad15) -> /Nodes/~RESET
- J11 pad 16: Net-(J11-Pad16) -> /Nodes/~READY_3
- J11 pad 17: Net-(J11-Pad17) -> /Nodes/~READY_4
- J11 pad 18: Net-(J11-Pad18) -> GND
- J11 pad 2: /Nodes/~RESET -> GND
- J11 pad 3: /Nodes/~CS1 -> /FPGA_CDONE
- J11 pad 4: /Nodes/SCK1 -> /Nodes/CRESETB
- J11 pad 5: /Nodes/SDO1_5 -> GND
- J11 pad 6: /Nodes/~READY_6 -> /Nodes/SCK0
- J11 pad 7: Net-(J11-Pad7) -> /Nodes/~CS0
- J11 pad 8: Net-(J11-Pad8) -> /Nodes/COPI0
- J11 pad 9: Net-(J11-Pad9) -> GND
- J12 pad 1: /Nodes/~CS0 -> +5V
- J12 pad 10: Net-(J12-Pad10) -> /Nodes/SCK1
- J12 pad 11: Net-(J12-Pad11) -> /Nodes/~CS1
- J12 pad 12: Net-(J12-Pad12) -> /Nodes/SDO1_6
- J12 pad 13: Net-(J12-Pad13) -> /CIPO1
- J12 pad 14: Net-(J12-Pad14) -> GND
- J12 pad 15: Net-(J12-Pad15) -> /Nodes/~RESET
- J12 pad 16: Net-(J12-Pad16) -> /Nodes/~READY_7
- J12 pad 18: Net-(J12-Pad18) -> GND
- J12 pad 2: /Nodes/~RESET -> GND
- J12 pad 3: /Nodes/~CS1 -> /FPGA_CDONE
- J12 pad 4: /Nodes/SCK1 -> /Nodes/CRESETB
- J12 pad 5: /Nodes/SDO1_2 -> GND
- J12 pad 6: /Nodes/~READY_3 -> /Nodes/SCK0
- J12 pad 7: Net-(J12-Pad7) -> /Nodes/~CS0
- J12 pad 8: Net-(J12-Pad8) -> /Nodes/COPI0
- J12 pad 9: Net-(J12-Pad9) -> GND
- J6 pad 1: /Nodes/~CS0 -> +5V
- J6 pad 10: Net-(J6-Pad10) -> /Nodes/SCK1
- J6 pad 11: Net-(J6-Pad11) -> /Nodes/~CS1
- J6 pad 12: Net-(J6-Pad12) -> /Nodes/SDO1_3
- J6 pad 13: Net-(J6-Pad13) -> /Nodes/SDO1_4
- J6 pad 14: Net-(J6-Pad14) -> GND
- J6 pad 15: Net-(J6-Pad15) -> /Nodes/~RESET
- J6 pad 16: Net-(J6-Pad16) -> /Nodes/~READY_4
- J6 pad 17: Net-(J6-Pad17) -> /Nodes/~READY_5
- J6 pad 18: Net-(J6-Pad18) -> GND
- J6 pad 2: /Nodes/~RESET -> GND
- J6 pad 3: /Nodes/~CS1 -> /FPGA_CDONE
- J6 pad 4: /Nodes/SCK1 -> /Nodes/CRESETB
- J6 pad 5: /Nodes/COPI1 -> GND
- J6 pad 6: /FPGA_~READY~ -> /Nodes/SCK0
- J6 pad 7: Net-(J6-Pad7) -> /Nodes/~CS0
- J6 pad 8: Net-(J6-Pad8) -> /Nodes/COPI0
- J6 pad 9: Net-(J6-Pad9) -> GND
- J7 pad 1: /Nodes/~CS0 -> +5V
- J7 pad 10: Net-(J7-Pad10) -> /Nodes/SCK1
- J7 pad 11: Net-(J7-Pad11) -> /Nodes/~CS1
- J7 pad 12: Net-(J7-Pad12) -> /Nodes/SDO1_0
- J7 pad 13: Net-(J7-Pad13) -> /Nodes/SDO1_1
- J7 pad 14: Net-(J7-Pad14) -> GND
- J7 pad 15: Net-(J7-Pad15) -> /Nodes/~RESET
- J7 pad 16: Net-(J7-Pad16) -> /Nodes/~READY_1
- J7 pad 17: Net-(J7-Pad17) -> /Nodes/~READY_2
- J7 pad 18: Net-(J7-Pad18) -> GND
- J7 pad 2: /Nodes/~RESET -> GND
- J7 pad 3: /Nodes/~CS1 -> /FPGA_CDONE
- J7 pad 4: /Nodes/SCK1 -> /Nodes/CRESETB
- J7 pad 5: /Nodes/~READY_4 -> GND
- J7 pad 6: /Nodes/SDO1_3 -> /Nodes/SCK0
- J7 pad 7: Net-(J7-Pad7) -> /Nodes/~CS0
- J7 pad 8: Net-(J7-Pad8) -> /Nodes/COPI0
- J7 pad 9: Net-(J7-Pad9) -> GND
- J8 pad 1: /Nodes/~CS0 -> +5V
- J8 pad 10: Net-(J8-Pad10) -> /Nodes/SCK1
- J8 pad 11: Net-(J8-Pad11) -> /Nodes/~CS1
- J8 pad 12: Net-(J8-Pad12) -> /Nodes/SDO1_4
- J8 pad 13: Net-(J8-Pad13) -> /Nodes/SDO1_5
- J8 pad 14: Net-(J8-Pad14) -> GND
- J8 pad 15: Net-(J8-Pad15) -> /Nodes/~RESET
- J8 pad 16: Net-(J8-Pad16) -> /Nodes/~READY_5
- J8 pad 17: Net-(J8-Pad17) -> /Nodes/~READY_6
- J8 pad 18: Net-(J8-Pad18) -> GND
- J8 pad 2: /Nodes/~RESET -> GND
- J8 pad 3: /Nodes/~CS1 -> /FPGA_CDONE
- J8 pad 4: /Nodes/SCK1 -> /Nodes/CRESETB
- J8 pad 5: /Nodes/SDO1_0 -> GND
- J8 pad 6: /Nodes/~READY_1 -> /Nodes/SCK0
- J8 pad 7: Net-(J8-Pad7) -> /Nodes/~CS0
- J8 pad 8: Net-(J8-Pad8) -> /Nodes/COPI0
- J8 pad 9: Net-(J8-Pad9) -> GND
- J9 pad 1: /Nodes/~CS0 -> +5V
- J9 pad 10: Net-(J9-Pad10) -> /Nodes/SCK1
- J9 pad 11: Net-(J9-Pad11) -> /Nodes/~CS1
- J9 pad 12: Net-(J9-Pad12) -> /Nodes/SDO1_1
- J9 pad 13: Net-(J9-Pad13) -> /Nodes/SDO1_2
- J9 pad 14: Net-(J9-Pad14) -> GND
- J9 pad 15: Net-(J9-Pad15) -> /Nodes/~RESET
- J9 pad 16: Net-(J9-Pad16) -> /Nodes/~READY_2
- J9 pad 17: Net-(J9-Pad17) -> /Nodes/~READY_3
- J9 pad 18: Net-(J9-Pad18) -> GND
- J9 pad 2: /Nodes/~RESET -> GND
- J9 pad 3: /Nodes/~CS1 -> /FPGA_CDONE
- J9 pad 4: /Nodes/SCK1 -> /Nodes/CRESETB
- J9 pad 5: /Nodes/SDO1_4 -> GND
- J9 pad 6: /Nodes/~READY_5 -> /Nodes/SCK0
- J9 pad 7: Net-(J9-Pad7) -> /Nodes/~CS0
- J9 pad 8: Net-(J9-Pad8) -> /Nodes/COPI0
- J9 pad 9: Net-(J9-Pad9) -> GND
- R21 pad 1: Net-(J1-Pad18) -> Net-(R21-Pad1)
- R25 pad 2: Net-(J13-Pad26) -> Net-(J12-Pad17)
Routing:
- net /USB_D-: track 260.9 -> 2.60 mm
- net /USB_D+: track 260.4 -> 2.63 mm
- net +5V: track 393.6 -> 140.6 mm
- net +12V: track 0.00 -> 197.1 mm
- net /CIPO1: track 2.86 -> 130.1 mm
- net +3V3: track 130.3 -> 9.75 mm
- net Net-(J1-Pad18): track 93.0 -> 0.00 mm
- net /~ETH_LEDL: track 69.3 -> 0.00 mm, vias 2 -> 0
- net Net-(J1-Pad20): track 61.3 -> 0.00 mm, vias 1 -> 0
- net /Nodes/COPI0: track 55.6 -> 9.67 mm
- net /SCK1: track 6.34 -> 49.1 mm
- net /~CS1: track 5.80 -> 48.5 mm, vias 2 -> 4
- net /COPI1: track 6.47 -> 47.1 mm
- net /Nodes/SCK0: track 48.8 -> 9.67 mm
- net Earth: track 38.1 -> 0.00 mm
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Other:
- board size 360 x 40 mm -> 250 x 40 mm

Commit message: Yet another rework in progress.
Parts:
- removed C6, C7: 1u, Capacitor_SMD:C_0402_1005Metric
- removed D2: PI_PWR, LED_SMD:LED_0603_1608Metric
- removed FB1: FB, Inductor_SMD:L_0805_2012Metric
- removed H1, H2, H3, H4: M3_MH, MountingHole:MountingHole_3.2mm_M3_DIN965_Pad
- removed J10: Node 6, Connector_PinHeader_2.00mm:PinHeader_1x18_P2.00mm_Vertical_SMD_Pin1Left
- removed J11: Node 3, Connector_PinHeader_2.00mm:PinHeader_1x18_P2.00mm_Vertical_SMD_Pin1Left
- removed J12: Node 7, Connector_PinHeader_2.00mm:PinHeader_1x18_P2.00mm_Vertical_SMD_Pin1Left
- removed J8: Node 5, Connector_PinHeader_2.00mm:PinHeader_1x18_P2.00mm_Vertical_SMD_Pin1Left
- removed J9: Node 2, Connector_PinHeader_2.00mm:PinHeader_1x18_P2.00mm_Vertical_SMD_Pin1Left
- removed OSHW2: Logo_Open_Hardware_Small, Symbol:OSHW-Symbol_8.9x8mm_Copper
- removed R13, R14, R15, R18, R21, R22, R25, R5, R9: 1k0, Resistor_SMD:R_0402_1005Metric
- removed R16, R19: 5k1, Resistor_SMD:R_0402_1005Metric
- removed R17, R26, R27, R28, R29, R30: 22R, Resistor_SMD:R_0402_1005Metric
- removed R39, R40, R41, R42, R43, R44, R45, R7: DNP, Resistor_SMD:R_0402_1005Metric
- removed U4: SN74LVC1G14DBV, Package_TO_SOT_SMD:SOT-23-5
- added C2: 47u, Capacitor_SMD:CP_Elec_6.3x5.9, F.Cu at (92.0, 19.0)
- added C5: 22u, Capacitor_SMD:C_0603_1608Metric, F.Cu at (126.6, 44.6)
- added D3: 5V, LED_SMD:LED_0603_1608Metric, F.Cu at (126.6, 47.3)
- added JP1: ~WL_nDisable, jkiv-library:J_Small_NC, F.Cu at (126.6, 58.7)
- added JP2: ~BT_nDisable, jkiv-library:J_Small_NC, F.Cu at (126.6, 4.74)
- added JP3: EEPROM_nWP, jkiv-library:J_Small_NC, F.Cu at (126.6, 53.3)
- added JP4: ~WL_nDisable, jkiv-library:J_Small_NC, F.Cu at (126.6, 41.9)
- added L2: 2.2u, Inductor_SMD:L_1008_2520Metric, F.Cu at (-130.0, 17.0)
- added OSHW1: Logo_Open_Hardware_Small, Symbol:OSHW-Symbol_8.9x8mm_Copper, F.Cu at (101.0, 42.5)
- added RN1: 22R, Resistor_SMD:R_Array_Convex_4x0603, F.Cu at (-99.0, 39.0)
- added RN2: 22R, Resistor_SMD:R_Array_Convex_4x0603, F.Cu at (-86.0, 39.0)
- added RN3: 22R, Resistor_SMD:R_Array_Convex_4x0603, F.Cu at (-105.0, 39.0)
- added RN4: 22R, Resistor_SMD:R_Array_Convex_4x0603, F.Cu at (-92.0, 39.0)
- added U2: TPS62140, Package_DFN_QFN:VQFN-16-1EP_3x3mm_P0.5mm_EP1.68x1.68mm_ThermalVias, F.Cu at (-130.0, 21.0)
- C3: value 1u -> 10u; footprint Capacitor_SMD:C_0402_1005Metric -> Capacitor_SMD:C_0603_1608Metric
- C4: value 1u -> 3.3n
- D1: value ACT_LED -> PI_ACT
- D4: value TPD2EUSB30DRTR -> 3v3; footprint digikey-footprints:SOT-3 -> LED_SMD:LED_0603_1608Metric
- J1: value Abracon_ARJ139 -> microSD; footprint jkiv-library:RJ45_Abracon_ARJ136 -> Connector_Card:microSD_HC_Molex_104031-0811; moved to B.Cu
- J2: value USB2.0 Type-C -> PWR; footprint Connector_USB:USB_C_Receptacle_Palconn_UTC16-G -> Connector_Molex:Molex_Mini-Fit_Jr_5569-04A2_2x02_P4.20mm_Horizontal
- J3: value Micro_SD_Card -> Abracon_ARJM11-502; footprint Connector_Card:microSD_HC_Molex_104031-0811 -> Connector_RJ:RJ45_Abracon_ARJP11A-MA_Horizontal; moved to F.Cu
- J4: value DP1435 PoE Module -> S; footprint jkiv-library:DP1435_Module -> Connector_PinHeader_1.27mm:PinHeader_1x20_P1.27mm_Vertical
- J5: value Node 0 -> E; footprint Connector_PinHeader_2.00mm:PinHeader_1x18_P2.00mm_Vertical_SMD_Pin1Left -> Connector_PinHeader_1.27mm:PinHeader_1x16_P1.27mm_Vertical
- J6: value Node 4 -> W; footprint Connector_PinHeader_2.00mm:PinHeader_1x18_P2.00mm_Vertical_SMD_Pin1Left -> Connector_PinHeader_1.27mm:PinHeader_1x16_P1.27mm_Vertical
- J7: value Node 1 -> N; footprint Connector_PinHeader_2.00mm:PinHeader_1x18_P2.00mm_Vertical_SMD_Pin1Left -> Connector_PinHeader_1.27mm:PinHeader_1x08_P1.27mm_Vertical
- R1: value 22R -> 220R
- R10, R11: value DNP -> 1k0
- R12: value DNP -> 100k
- R2: value 22R -> 1k0
- R3, R4: value 1k0 -> 220R
- R6: value DNP -> 330R
- R8: value DNP -> 220R
- U1: value Compute_Module_4_Functional -> CM4
- moved J3 248.0 mm to (-121.0, 32.0), turned to 270 degrees
- moved J6 230.5 mm to (-37.0, 13.6), turned to 270 degrees
- moved U1 206.5 mm to (-91.0, 30.0), turned to 270 degrees
- moved J5 205.3 mm to (-56.0, 47.6), turned to 90 degrees
- moved J7 195.4 mm to (-34.5, 31.6)
- moved J2 175.8 mm to (95.7, 27.9), turned to 270 degrees
- moved D4 143.7 mm to (126.6, 14.1), turned to 0 degrees
- moved J1 143.5 mm to (-96.0, 58.0), turned to 0 degrees
- moved C1 135.0 mm to (126.6, 50.4)
- moved J4 133.9 mm to (-58.5, 21.5), turned to 0 degrees
- moved R3 108.7 mm to (126.6, -0.63)
- moved R4 100.5 mm to (126.6, 7.16)
- moved R6 94.4 mm to (126.6, 11.6)
- moved D7 90.1 mm to (126.6, 1.95), turned to 0 degrees
- moved R8 87.2 mm to (126.6, 18.9)
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Connections:
- net /SD_PON renamed /SD_PWR_ON
- net /THERM_1W renamed Net-(U1-Pad54)
- net /~nRPIBOOT renamed /~PI_nRPIBOOT
- C1 pad 1: /USB_VBUS -> +3V3
- C3 pad 1: +3V3 -> GND
- C3 pad 2: GND -> VBUS
- C4 pad 1: +3V3 -> Net-(C4-Pad1)
- D4 pad 1: /USB_D+ -> Net-(D4-Pad1)
- D4 pad 2: /USB_D- -> +3V3
- J1 pad 1: /ETH_CT -> /SD_DAT2
- J1 pad 10: /ETH_TD1- -> (no net)
- J1 pad 11: /ETH_TD1+ -> (no net)
- J1 pad 2: /ETH_TD3- -> /SD_DAT3
- J1 pad 3: /ETH_TD3+ -> /SD_CMD
- J1 pad 4: /ETH_TD2+ -> +3V3
- J1 pad 5: /ETH_TD2- -> /SD_CLK
- J1 pad 6: /ETH_CT -> GND
- J1 pad 7: /ETH_CT -> /SD_DAT0
- J1 pad 8: /ETH_TD4+ -> /SD_DAT1
- J1 pad 9: /ETH_TD4- -> GND
- J3 pad 1: /SD_DAT2 -> /ETH_TD1+
- J3 pad 10: (no net) -> /ETH_TD4-
- J3 pad 11: (no net) -> +3V3
- J3 pad 2: /SD_DAT3 -> /ETH_TD1-
- J3 pad 3: /SD_CMD -> /ETH_TD2+
- J3 pad 4: +3V3 -> /ETH_TD2-
- J3 pad 5: /SD_CLK -> Net-(J3-Pad5)
- J3 pad 6: GND -> Net-(J3-Pad5)
- J3 pad 7: /SD_DAT0 -> /ETH_TD3+
- J3 pad 9: Net-(J3-Pad9) -> /ETH_TD4+
- J4 pad 1: /PoE_TAP1 -> GND
- J4 pad 2: /PoE_TAP2 -> /FPGA_~READY~
- J4 pad 3: /PoE_TAP3 -> GND
- J4 pad 4: /PoE_TAP4 -> /Nodes/SCK1
- J4 pad 5: +12V -> GND
- J4 pad 6: GND -> /Nodes/COPI1
- J5 pad 1: +5V -> GND
- J5 pad 10: GND -> Net-(J5-Pad10)
- J5 pad 11: /Nodes/~CS1 -> GND
- J5 pad 12: /Nodes/SDO1_0 -> Net-(J5-Pad12)
- J5 pad 13: /Nodes/COPI1 -> GND
- J5 pad 14: /Nodes/SCK1 -> Net-(J5-Pad14)
- J5 pad 16: /FPGA_CDONE -> Net-(J5-Pad16)
- J5 pad 3: /FPGA_~READY~ -> GND
- J5 pad 4: /Nodes/~READY_1 -> GND
- J5 pad 5: /Nodes/~RESET -> GND
- J5 pad 7: /Nodes/COPI0 -> GND
- J5 pad 8: /Nodes/~CS0 -> GND
- J5 pad 9: /Nodes/SCK0 -> GND
- J6 pad 1: +5V -> GND
- J6 pad 10: /Nodes/SCK1 -> GND
- J6 pad 11: /Nodes/~CS1 -> GND
- J6 pad 12: /Nodes/SDO1_3 -> GND
- J6 pad 13: /Nodes/SDO1_4 -> VBUS
- J6 pad 14: GND -> VBUS
- J6 pad 15: /Nodes/~RESET -> VBUS
- J6 pad 16: /Nodes/~READY_4 -> VBUS
- J6 pad 3: /FPGA_CDONE -> GND
- J6 pad 4: /Nodes/CRESETB -> GND
- J6 pad 6: /Nodes/SCK0 -> GND
- J6 pad 7: /Nodes/~CS0 -> GND
- J6 pad 8: /Nodes/COPI0 -> GND
- J7 pad 1: +5V -> /Nodes/~CS1_0
- J7 pad 3: /FPGA_CDONE -> /Nodes/SDO1_0
- J7 pad 4: /Nodes/CRESETB -> GND
- J7 pad 5: GND -> /Nodes/SCK1_0
- J7 pad 6: /Nodes/SCK0 -> GND
- J7 pad 7: /Nodes/~CS0 -> /Nodes/~READY_1
- J7 pad 8: /Nodes/COPI0 -> GND
- R1 pad 1: /Nodes/SCK0 -> Net-(D1-Pad1)
- R1 pad 2: /SCK0 -> /PI_LED_nACT
- R10 pad 1: GND -> Net-(J3-Pad14)
- R10 pad 2: /CM4_EN -> /~ETH_LEDR
- R11 pad 1: GND -> Net-(J3-Pad12)
- R11 pad 2: /RUN_PG -> /~ETH_LEDL
- R12 pad 1: GND -> +5V
- R12 pad 2: /~nEXTRST -> Net-(R12-Pad2)
- R2 pad 1: /Nodes/COPI0 -> GND
- R2 pad 2: /COPI0 -> /Nodes/node5/~READY_IN
- R3 pad 1: /CM4_EN -> Net-(R3-Pad1)
- R3 pad 2: +3V3 -> /PI_nRPI_BOOT
- R4 pad 1: /RUN_PG -> Net-(R4-Pad1)
- R4 pad 2: +3V3 -> /PI_GLOBAL_EN
- R6 pad 1: /WL_EN -> Net-(D3-Pad1)
- R6 pad 2: +3V3 -> GND
- R8 pad 1: /EEPROM_WE -> Net-(D4-Pad1)
- R8 pad 2: +3V3 -> GND
- U1 pad 100: /~nEXTRST -> Net-(U1-Pad100)
- U1 pad 101: Net-(U1-Pad101) -> (no net)
- U1 pad 103: /USB_D- -> (no net)
- U1 pad 105: /USB_D+ -> (no net)
- U1 pad 20: /EEPROM_WE -> Net-(JP3-Pad2)
- U1 pad 21: /~LED_ACT -> /PI_LED_nACT
- U1 pad 89: /WL_EN -> Net-(JP1-Pad2)
- U1 pad 91: /BT_EN -> Net-(JP2-Pad2)
- U1 pad 92: /RUN_PG -> Net-(U1-Pad92)
- U1 pad 95: /~PI_LED_nPWR -> /PI_LED_nPWR
- U1 pad 99: /CM4_EN -> /PI_GLOBAL_EN
Routing:
- net +12V: track 197.1 -> 0.00 mm
- net +5V: track 140.6 -> 0.00 mm
- net /CIPO1: track 130.1 -> 0.00 mm
- net GND: track 114.7 -> 0.00 mm, vias 66 -> 0
- net /ETH_TD2-: track 67.7 -> 0.00 mm, vias 2 -> 0
- net /ETH_TD3-: track 67.3 -> 0.00 mm
- net /ETH_TD3+: track 67.0 -> 0.00 mm
- net /ETH_TD2+: track 66.6 -> 0.00 mm, vias 2 -> 0
- net /ETH_TD1-: track 65.9 -> 0.00 mm
- net /ETH_TD1+: track 65.6 -> 0.00 mm
- net /ETH_TD4+: track 62.8 -> 0.00 mm
- net /ETH_TD4-: track 62.5 -> 0.00 mm
- net /SCK1: track 49.1 -> 0.00 mm, vias 2 -> 0
- net /~CS1: track 48.5 -> 0.00 mm, vias 4 -> 0
- net /COPI1: track 47.1 -> 0.00 mm, vias 2 -> 0
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- removed copper zone on B.Cu, net GND
Other:
- outline, holes or cut-outs redrawn
